File: docs/leo/shared_memory.kicad_sch (KiCad schematic)
At the start: 9 parts, among them IC15 MB81C78A, IC16 MB81C78A, IC17 74153, IC18 74153, IC19 74153, IC25 74153, IC26 74153, IC27 74153, IC28 74153

Commit message: Additional schematic updates
Parts:
- added IC10, IC9: 74LS273, symbol 74xx:74LS273
- added IC22, IC23: 74LS245, symbol 74xx:74LS245
- added IC30, IC31: 74LS374, symbol 74xx:74LS374
Connections:
- net ~{MEM_WR}: now also IC22.1 (A->B), IC23.1 (A->B)
- net SHARED_D0 renamed D0
- net D0: now also IC22.9 (A7), IC30.2 (O0)
- net SHARED_D1 renamed D1
- net D1: now also IC22.8 (A6), IC30.5 (O1)
- net SHARED_D10 renamed D10
- net D10: now also IC23.7 (A5), IC31.6 (O2)
- net SHARED_D11 renamed D11
- net D11: now also IC23.6 (A4), IC31.9 (O3)
- net SHARED_D12 renamed D12
- net D12: now also IC23.5 (A3), IC31.12 (O4)
- net SHARED_D13 renamed D13
- net D13: now also IC23.4 (A2), IC31.15 (O5)
- net SHARED_D14 renamed D14
- net D14: now also IC23.3 (A1), IC31.16 (O6)
- net SHARED_D15 renamed D15
- net D15: now also IC23.2 (A0), IC31.19 (O7)
- net SHARED_D2 renamed D2
- net D2: now also IC22.7 (A5), IC30.6 (O2)
- net SHARED_D3 renamed D3
- net D3: now also IC22.6 (A4), IC30.9 (O3)
- net SHARED_D4 renamed D4
- net D4: now also IC22.5 (A3), IC30.12 (O4)
- net SHARED_D5 renamed D5
- net D5: now also IC22.4 (A2), IC30.15 (O5)
- net SHARED_D6 renamed D6
- net D6: now also IC22.3 (A1), IC30.16 (O6)
- net SHARED_D7 renamed D7
- net D7: now also IC22.2 (A0), IC30.19 (O7)
- net SHARED_D8 renamed D8
- net D8: now also IC23.9 (A7), IC31.2 (O0)
- net SHARED_D9 renamed D9
- net D9: now also IC23.8 (A6), IC31.5 (O1)
- new net BUF_D0: IC22.11 (B7)
- new net BUF_D1: IC22.12 (B6)
- new net BUF_D10: IC23.13 (B5)
- new net BUF_D11: IC23.14 (B4)
- new net BUF_D12: IC23.15 (B3)
- new net BUF_D13: IC23.16 (B2)
- new net BUF_D14: IC23.17 (B1)
- new net BUF_D15: IC23.18 (B0)
- new net BUF_D2: IC22.13 (B5)
- new net BUF_D3: IC22.14 (B4)
- new net BUF_D4: IC22.15 (B3)
- new net BUF_D5: IC22.16 (B2)
- new net BUF_D6: IC22.17 (B1)
- new net BUF_D7: IC22.18 (B0)
- new net BUF_D8: IC23.11 (B7)
- new net BUF_D9: IC23.12 (B6)
- new net IC42_103: IC30.11 (Cp), IC31.11 (Cp)
- new net IC42_131: IC30.1 (OE), IC31.1 (OE)
- new net IC42_136: IC22.19 (CE), IC23.19 (CE)
