File: docs/leo/audio_cpu.kicad_sch (KiCad schematic)
At the start: 20 parts, among them IC1 74LS04, IC14 High ROM, IC17 Low ROM, IC2 V35S, IC41 74LS244, IC5 74LS373, IC50 74LS245, IC6 74LS373, X1 14.31818Mhz

Commit message: B Board Audio section complete
Parts:
- removed IC13, IC21: (no value), symbol 74xx:74LS74
- added IC8: Sample ROM, symbol Memory_EPROM:27C080
- added J1, J2: Jumper_3_Bridged12, symbol Jumper:Jumper_3_Bridged12
- gave numbers to parts that had none: 1
Connections:
- net A0 is gone; now on net A1: IC14.12 (A0), IC15.10 (A0), IC16.10 (A0), IC17.12 (A0), IC2.30 (A9/A1), IC41.8 (I3a), IC6.8 (D3)
- net A1: no longer IC14.11 (A1), IC15.9 (A1), IC16.9 (A1), IC17.11 (A1), IC2.31 (A10/A2), IC41.13 (I1b), IC6.13 (D4)
- net A10: now also IC14.26 (A9), IC15.24 (A9), IC16.24 (A9), IC17.26 (A9), IC6.12 (O4); no longer IC14.23 (A10), IC15.21 (A10), IC16.21 (A10), IC17.23 (A10), IC6.6 (O2)
- net A11: now also IC14.23 (A10), IC15.21 (A10), IC16.21 (A10), IC17.23 (A10), IC6.6 (O2); no longer IC14.25 (A11), IC15.23 (A11), IC16.23 (A11), IC17.25 (A11), IC6.5 (O1)
- net A12: now also IC14.25 (A11), IC15.23 (A11), IC16.23 (A11), IC17.25 (A11), IC6.5 (O1); no longer IC14.4 (A12), IC15.2 (A12), IC16.2 (A12), IC17.4 (A12), IC6.15 (O5)
- net A13: now also IC14.4 (A12), IC15.2 (A12), IC16.2 (A12), IC17.4 (A12), IC6.15 (O5); no longer IC14.28 (A13), IC17.28 (A13), IC6.16 (O6)
- net A14: now also IC14.28 (A13), IC17.28 (A13), IC6.16 (O6); no longer IC14.29 (A14), IC17.29 (A14), IC6.2 (O0)
- net A15: now also IC14.29 (A14), IC17.29 (A14), IC6.2 (O0), U?.5 (I5); no longer IC14.3 (A15), IC17.3 (A15), IC6.19 (O7)
- net A16: now also IC14.3 (A15), IC17.3 (A15), IC6.19 (O7), U?.4 (I4); no longer IC14.2 (A16), IC17.2 (A16), IC5.9 (O3)
- net A17: now also IC14.2 (A16), IC17.2 (A16), IC5.9 (O3), U?.3 (I3); no longer IC14.30 (A17), IC17.30 (A17), IC5.12 (O4)
- net A18: now also IC14.30 (A17), IC17.30 (A17), IC5.12 (O4), U?.2 (I2); no longer IC14.31 (A18), IC17.31 (A18), IC5.6 (O2)
- net A19: now also IC14.31 (A18), IC17.31 (A18), IC5.6 (O2), U?.1 (I1); no longer IC14.1 (A19), IC17.1 (A19)
- net A2: now also IC14.11 (A1), IC15.9 (A1), IC16.9 (A1), IC17.11 (A1), IC2.31 (A10/A2), IC41.13 (I1b), IC6.13 (D4); no longer IC14.10 (A2), IC15.8 (A2), IC16.8 (A2), IC17.10 (A2), IC2.32 (A11/A3), IC41.6 (I2a), IC6.7 (D2)
- net A3: now also IC14.10 (A2), IC15.8 (A2), IC16.8 (A2), IC17.10 (A2), IC2.32 (A11/A3), IC41.6 (I2a), IC6.7 (D2); no longer IC14.9 (A3), IC15.7 (A3), IC16.7 (A3), IC17.9 (A3), IC2.33 (A12/A4), IC41.4 (I1a), IC6.4 (D1)
- net A4: now also IC14.9 (A3), IC15.7 (A3), IC16.7 (A3), IC17.9 (A3), IC2.33 (A12/A4), IC41.4 (I1a), IC6.4 (D1); no longer IC14.8 (A4), IC15.6 (A4), IC16.6 (A4), IC17.8 (A4), IC2.34 (A13/A5), IC41.15 (I2b), IC6.14 (D5)
- net A5: now also IC14.8 (A4), IC15.6 (A4), IC16.6 (A4), IC17.8 (A4), IC2.34 (A13/A5), IC41.15 (I2b), IC6.14 (D5); no longer IC14.7 (A5), IC15.5 (A5), IC16.5 (A5), IC17.7 (A5), IC2.35 (A14/A6), IC41.17 (I3b), IC6.17 (D6)
- net A6: now also IC14.7 (A5), IC15.5 (A5), IC16.5 (A5), IC17.7 (A5), IC2.35 (A14/A6), IC41.17 (I3b), IC6.17 (D6); no longer IC14.6 (A6), IC15.4 (A6), IC16.4 (A6), IC17.6 (A6), IC2.36 (A15/A7), IC41.2 (I0a), IC6.3 (D0)
- net A7: now also IC14.6 (A6), IC15.4 (A6), IC16.4 (A6), IC17.6 (A6), IC2.36 (A15/A7), IC41.2 (I0a), IC6.3 (D0); no longer IC14.5 (A7), IC15.3 (A7), IC16.3 (A7), IC17.5 (A7), IC2.37 (A16/A8), IC6.18 (D7)
- net A8: now also IC14.5 (A7), IC15.3 (A7), IC16.3 (A7), IC17.5 (A7), IC2.37 (A16/A8), IC6.18 (D7); no longer IC14.27 (A8), IC15.25 (A8), IC16.25 (A8), IC17.27 (A8), IC6.9 (O3)
- net A9: now also IC14.27 (A8), IC15.25 (A8), IC16.25 (A8), IC17.27 (A8), IC6.9 (O3); no longer IC14.26 (A9), IC15.24 (A9), IC16.24 (A9), IC17.26 (A9), IC6.12 (O4)
- net D0: now also IC2.13 (D0)
- net D1: now also IC2.14 (D1)
- net D10: now also IC2.23 (D10)
- net D11: now also IC2.24 (D11)
- net D12: now also IC2.25 (D12)
- net D13: now also IC2.26 (D13)
- net D14: now also IC2.27 (D14)
- net D15: now also IC2.28 (D15)
- net D2: now also IC2.15 (D2)
- net D3: now also IC2.16 (D3)
- net D4: now also IC2.17 (D4)
- net D5: now also IC2.18 (D5)
- net D6: now also IC2.19 (D6)
- net D7: now also IC2.20 (D7)
- net D8: now also IC2.21 (D8)
- net D9: now also IC2.22 (D9)
- net GND: now also IC22.5, IC8.16 (GND), IC8.22 (~{CE}), IC8.24 (~{OE}), J1.1 (A), J2.1 (A)
- net V35_PULLDN: now also IC2.59 (P10/NMA); no longer IC2.3 (IC)
- net V35_PULLUP: now also IC2.10 (P05), IC2.11 (P06), IC2.4 (P00), IC2.43 (~{CTS0}), IC2.46 (~{CTS1}), IC2.5 (P01), IC2.6 (P02), IC2.62 (P13/~{INTP2}/~{INTAK}), IC2.63 (P14/INT/~{POLL}), IC2.64 (P15/TOUT), IC2.65 (P16/~{SCK0}), IC2.66 (P17/READY), IC2.7 (P03), IC2.8 (P04), J1.3 (B), J2.3 (B)
- net VCC: now also IC4.1 (~{R}), IC4.10 (~{S}), IC4.13 (~{R}), IC4.4 (~{S}), IC8.32 (VCC)
- net at IC14.24 (~{OE}), IC15.22 (~{OE}), IC16.22 (~{OE})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: now also IC22.4
- net ~{SND_OE}: now reaches IC22.6
- net ~{RAM_CS}: now reaches IC22.13, IC22.2, U?.15 (IO5)
- net ~{W_STB}: now reaches IC15.27 (~{WE}), IC16.27 (~{WE}), IC18.8, IC41.11 (I0b), U?.9 (I9)
- net ~{ROM_CS}: now reaches IC14.22 (~{CE}), IC17.22 (~{CE}), U?.13 (IO7)
- net ~{MREQ}: now reaches U?.6 (I6)
- net ~{MREQ}: now also IC3.6, IC5.11 (LE), IC6.11 (LE)
- net SND_A0: now reaches IC41.12 (O3a)
- net SND_A2: now reaches IC41.14 (O2a)
- net SND_A3: now reaches IC41.16 (O1a)
- net SND_A6: now reaches IC41.18 (O0a)
- net SND_A5: now reaches IC41.3 (O3b)
- net SND_A4: now reaches IC41.5 (O2b)
- net SND_A1: now reaches IC41.7 (O1b)
- net ~{SND_W}: now reaches IC41.9 (O0b)
- net at IC1.12, IC1.3: now also IC4.11 (C)
- net SND_D7: now reaches IC50.11 (B7), RA3.9 (R8)
- net SND_D6: now reaches IC50.12 (B6), RA3.8 (R7)
- net SND_D5: now reaches IC50.13 (B5), RA3.7 (R6)
- net SND_D4: now reaches IC50.14 (B4), RA3.6 (R5)
- net SND_D3: now reaches IC50.15 (B3), RA3.5 (R4)
- net SND_D2: now reaches IC50.16 (B2), RA3.4 (R3)
- net SND_D1: now reaches IC50.17 (B1), RA3.3 (R2)
- net SND_D0: now reaches IC50.18 (B0), RA3.2 (R1)
- net at IC4.12 (D): now also IC4.8 (~{Q})
- net at IC4.9 (Q): now also IC4.3 (C)
- net at IC2.53 (N/~{S}): now also J2.2 (C)
- net ~{RESET}: now reaches IC2.81 (~{RESET})
- net at IC4.2 (D): now also IC4.6 (~{Q})
- net CLK_3_57: now reaches IC4.5 (Q)
- net CN3_A16 renamed ~{SND_INTP0}
- net CN3_B15 renamed ~{SND_INTP1}
- net CN3_B16 renamed ~{SND_CS}
- new net: IC2.3 (IC), J1.2 (C)
- new net A20: IC14.1 (A19), IC17.1 (A19)
- new net SAMP_A0: IC8.12 (A0)
- new net SAMP_A1: IC8.11 (A1)
- new net SAMP_A10: IC8.23 (A10)
- new net SAMP_A11: IC8.25 (A11)
- new net SAMP_A12: IC8.4 (A12)
- new net SAMP_A13: IC8.28 (A13)
- new net SAMP_A14: IC8.29 (A14)
- new net SAMP_A15: IC8.3 (A15)
- new net SAMP_A16: IC8.2 (A16)
- new net SAMP_A17: IC8.30 (A17)
- new net SAMP_A18: IC8.31 (A18)
- new net SAMP_A19: IC8.1 (A19)
- new net SAMP_A2: IC8.10 (A2)
- new net SAMP_A3: IC8.9 (A3)
- new net SAMP_A4: IC8.8 (A4)
- new net SAMP_A5: IC8.7 (A5)
- new net SAMP_A6: IC8.6 (A6)
- new net SAMP_A7: IC8.5 (A7)
- new net SAMP_A8: IC8.27 (A8)
- new net SAMP_A9: IC8.26 (A9)
- new net SAMP_D0: IC8.13 (D0)
- new net SAMP_D1: IC8.14 (D1)
- new net SAMP_D2: IC8.15 (D2)
- new net SAMP_D3: IC8.17 (D3)
- new net SAMP_D4: IC8.18 (D4)
- new net SAMP_D5: IC8.19 (D5)
- new net SAMP_D6: IC8.20 (D6)
- new net SAMP_D7: IC8.21 (D7)
- no-connect marks 0 -> 6
Other:
- moved on the sheet: IC14, IC15, IC16, IC17, IC18A, IC18B, IC18C, IC18D, IC1A, IC1B, IC1C, IC1D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

Commit message: Finished GA20 pinout Roughed in sound latch, ym2151 and ga20 signals in A board
Parts:
- IC15, IC16: value (none) -> CXK5863; footprint (none) -> Package_DIP:DIP-28_W15.24mm
- IC18: value (none) -> 74LS00
- IC22: value (none) -> 74LS32
- IC3: value (none) -> 74LS04
- IC4: value (none) -> 74LS74
- U?: value (none) -> PAL16L8
Connections:
- net SND_A0 is gone; now on net SND_A1: IC41.12 (O3a)
- net SND_A1: no longer IC41.7 (O1b)
- net SND_A2: now also IC41.7 (O1b); no longer IC41.14 (O2a)
- net SND_A3: now also IC41.14 (O2a); no longer IC41.16 (O1a)
- net SND_A4: now also IC41.16 (O1a); no longer IC41.5 (O2b)
- net SND_A5: now also IC41.5 (O2b); no longer IC41.3 (O3b)
- net SND_A6: now also IC41.3 (O3b); no longer IC41.18 (O0a)
- new net SND_A7: IC41.18 (O0a)
Changed lines of the file:
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@@
     )
   )
-  (global_label "SND_A0" (shape output) (at 462.28 254 0) (fields_autoplaced)
+  (global_label "SND_A1" (shape output) (at 462.28 254 0) (fields_autoplaced)
     (effects (font (size 1.27 1.27)) (justify left))
     (property "Intersheet References" "${INTERSHEET_REFS}" (id 0) (at 471.7688 253.9206 0)
@@
     )
   )
-  (global_label "SND_A6" (shape output) (at 462.28 246.38 0) (fields_autoplaced)
+  (global_label "SND_A7" (shape output) (at 462.28 246.38 0) (fields_autoplaced)
     (effects (font (size 1.27 1.27)) (justify left))
     (property "Intersheet References" "${INTERSHEET_REFS}" (id 0) (at 471.7688 246.3006 0)
@@
     )
   )
-  (global_label "SND_A3" (shape output) (at 462.28 248.92 0) (fields_autoplaced)
+  (global_label "SND_A4" (shape output) (at 462.28 248.92 0) (fields_autoplaced)
     (effects (font (size 1.27 1.27)) (justify left))
     (property "Intersheet References" "${INTERSHEET_REFS}" (id 0) (at 471.7688 248.8406 0)
@@
     )
   )
-  (global_label "SND_A4" (shape output) (at 462.28 261.62 0) (fields_autoplaced)
+  (global_label "SND_A5" (shape output) (at 462.28 261.62 0) (fields_autoplaced)
     (effects (font (size 1.27 1.27)) (justify left))
     (property "Intersheet References" "${INTERSHEET_REFS}" (id 0) (at 471.7688 261.5406 0)
@@
     )
   )
-  (global_label "SND_A1" (shape output) (at 462.28 259.08 0) (fields_autoplaced)
+  (global_label "SND_A2" (shape output) (at 462.28 259.08 0) (fields_autoplaced)
     (effects (font (size 1.27 1.27)) (justify left))
     (property "Intersheet References" "${INTERSHEET_REFS}" (id 0) (at 471.7688 259.0006 0)
@@
     )
   )
-  (global_label "SND_A5" (shape output) (at 462.28 264.16 0) (fields_autoplaced)
+  (global_label "SND_A6" (shape output) (at 462.28 264.16 0) (fields_autoplaced)
     (effects (font (size 1.27 1.27)) (justify left))
     (property "Intersheet References" "${INTERSHEET_REFS}" (id 0) (at 471.7688 264.0806 0)
@@
     )
   )
-  (global_label "SND_A2" (shape output) (at 462.28 251.46 0) (fields_autoplaced)
+  (global_label "SND_A3" (shape output) (at 462.28 251.46 0) (fields_autoplaced)
     (effects (font (size 1.27 1.27)) (justify left))
     (property "Intersheet References" "${INTERSHEET_REFS}" (id 0) (at 471.7688 251.3806 0)
@@
     (in_bom yes) (on_board yes) (fields_autoplaced)
     (property "Reference" "IC3" (id 0) (at 715.01 133.35 0))
-    (property "Value" "" (id 1) (at 715.01 135.89 0))
+    (property "Value" "74LS04" (id 1) (at 715.01 135.89 0))
     (property "Footprint" "" (id 2) (at 715.01 142.24 0)
       (effects (font (size 1.27 1.27)) hide)
@@
     (in_bom yes) (on_board yes) (fields_autoplaced)
     (property "Reference" "IC22" (id 0) (at 687.07 170.18 0))
-    (property "Value" "" (id 1) (at 687.07 172.72 0))
+    (property "Value" "74LS32" (id 1) (at 687.07 172.72 0))
     (property "Footprint" "" (id 2) (at 687.07 179.07 0)
       (effects (font (size 1.27 1.27)) hide)
@@
     (in_bom yes) (on_board yes) (fields_autoplaced)
     (property "Reference" "IC18" (id 0) (at 262.89 237.49 0))
-    (property "Value" "" (id 1) (at 262.89 240.03 0))
+    (property "Value" "74LS00" (id 1) (at 262.89 240.03 0))
     (property "Footprint" "" (id 2) (at 262.89 246.38 0)
       (effects (font (size 1.27 1.27)) hide)
@@
     (in_bom yes) (on_board yes) (fields_autoplaced)
     (property "Reference" "IC3" (id 0) (at 180.34 111.76 0))
-    (property "Value" "" (id 1) (at 180.34 114.3 0))
+    (property "Value" "74LS04" (id 1) (at 180.34 114.3 0))
     (property "Footprint" "" (id 2) (at 180.34 120.65 0)
       (effects (font (size 1.27 1.27)) hide)
@@
     (in_bom yes) (on_board yes) (fields_autoplaced)
     (property "Reference" "IC22" (id 0) (at 293.37 234.95 0))
-    (property "Value" "" (id 1) (at 293.37 237.49 0))
+    (property "Value" "74LS32" (id 1) (at 293.37 237.49 0))
     (property "Footprint" "" (id 2) (at 293.37 243.84 0)
       (effects (font (size 1.27 1.27)) hide)
@@
       (effects (font (size 1.27 1.27)) (justify left))
     )
-    (property "Value" "" (id 1) (at 175.26 250.1899 90)
+    (property "Value" "74LS32" (id 1) (at 175.26 250.1899 90)
       (effects (font (size 1.27 1.27)) (justify left))
     )
@@
       (effects (font (size 1.27 1.27)) (justify left))
     )
-    (property "Value" "" (id 1) (at 137.9094 288.29 0)
-      (effects (font (size 1.27 1.27)) (justify left))
-    )
-    (property "Footprint" "" (id 2) (at 156.21 335.28 0)
+    (property "Value" "CXK5863" (id 1) (at 137.9094 288.29 0)
+      (effects (font (size 1.27 1.27)) (justify left))
+    )
+    (property "Footprint" "Package_DIP:DIP-28_W15.24mm" (id 2) (at 156.21 335.28 0)
       (effects (font (size 1.27 1.27)) hide)
     )
@@
     (in_bom yes) (on_board yes) (fields_autoplaced)
     (property "Reference" "IC18" (id 0) (at 685.8 149.86 0))
-    (property "Value" "" (id 1) (at 685.8 152.4 0))
+    (property "Value" "74LS00" (id 1) (at 685.8 152.4 0))
     (property "Footprint" "" (id 2) (at 685.8 158.75 0)
       (effects (font (size 1.27 1.27)) hide)
@@
       (effects (font (size 1.27 1.27)) (justify left))
     )
-    (property "Value" "" (id 1) (at 399.3006 242.57 0)
+    (property "Value" "PAL16L8" (id 1) (at 399.3006 242.57 0)
       (effects (font (size 1.27 1.27)) (justify left))
     )
@@
     (in_bom yes) (on_board yes)
     (property "Reference" "IC3" (id 0) (at 224.79 246.38 0))
-    (property "Value" "" (id 1) (at 224.79 248.92 0))
+    (property "Value" "74LS04" (id 1) (at 224.79 248.92 0))
     (property "Footprint" "" (id 2) (at 222.25 242.57 0)
       (effects (font (size 1.27 1.27)) hide)
@@
     (in_bom yes) (on_board yes)
     (property "Reference" "IC3" (id 0) (at 245.11 236.22 0))
-    (property "Value" "" (id 1) (at 245.11 238.76 0))
+    (property "Value" "74LS04" (id 1) (at 245.11 238.76 0))
     (property "Footprint" "" (id 2) (at 241.3 242.57 0)
       (effects (font (size 1.27 1.27)) hide)
@@
     (in_bom yes) (on_board yes)
     (property "Reference" "IC3" (id 0) (at 242.57 256.54 0))
-    (property "Value" "" (id 1) (at 242.57 259.08 0))
+    (property "Value" "74LS04" (id 1) (at 242.57 259.08 0))
     (property "Footprint" "" (id 2) (at 241.3 251.46 0)
       (effects (font (size 1.27 1.27)) hide)
@@
     (in_bom yes) (on_board yes) (fields_autoplaced)
     (property "Reference" "IC18" (id 0) (at 687.07 133.35 0))
-    (property "Value" "" (id 1) (at 687.07 135.89 0))
+    (property "Value" "74LS00" (id 1) (at 687.07 135.89 0))
     (property "Footprint" "" (id 2) (at 687.07 142.24 0)
       (effects (font (size 1.27 1.27)) hide)
@@
       (effects (font (size 1.27 1.27)) hide)
     )
-    (property "Value" "" (id 1) (at 151.13 226.06 0))
+    (property "Value" "GND" (id 1) (at 151.13 226.06 0))
     (property "Footprint" "" (id 2) (at 151.13 220.98 0)
       (effects (font (size 1.27 1.27)) hide)
@@
       (effects (font (size 1.27 1.27)) (justify left))
     )
-    (property "Value" "" (id 1) (at 365.76 181.61 0)
+    (property "Value" "74LS74" (id 1) (at 365.76 181.61 0)
       (effects (font (size 1.27 1.27)) (justify left))
     )
@@
       (effects (font (size 1.27 1.27)) (justify right))
     )
-    (property "Value" "" (id 1) (at 144.78 250.19 90)
+    (property "Value" "74LS32" (id 1) (at 144.78 250.19 90)
       (effects (font (size 1.27 1.27)) (justify right))
     )
@@
       (effects (font (size 1.27 1.27)) (justify left))
     )
-    (property "Value" "" (id 1) (at 402.59 181.61 0)
+    (property "Value" "74LS74" (id 1) (at 402.59 181.61 0)
       (effects (font (size 1.27 1.27)) (justify left))
     )
@@
     (in_bom yes) (on_board yes) (fields_autoplaced)
     (property "Reference" "IC18" (id 0) (at 262.89 270.51 0))
-    (property "Value" "" (id 1) (at 262.89 267.97 0))
+    (property "Value" "74LS00" (id 1) (at 262.89 267.97 0))
     (property "Footprint" "" (id 2) (at 262.89 261.62 0)
       (effects (font (size 1.27 1.27)) hide)
@@
     (in_bom yes) (on_board yes) (fields_autoplaced)
     (property "Reference" "IC3" (id 0) (at 165.1 111.76 0))
-    (property "Value" "" (id 1) (at 165.1 114.3 0))
+    (property "Value" "74LS04" (id 1) (at 165.1 114.3 0))
     (property "Footprint" "" (id 2) (at 165.1 120.65 0)
       (effects (font (size 1.27 1.27)) hide)
@@
       (effects (font (size 1.27 1.27)) (justify right))
     )
-    (property "Value" "" (id 1) (at 189.9794 287.02 0)
+    (property "Value" "CXK5863" (id 1) (at 189.9794 287.02 0)
       (effects (font (size 1.27 1.27)) (justify right))
     )
-    (property "Footprint" "" (id 2) (at 210.82 334.01 0)
-      (effects (font (size 1.27 1.27)) hide)
-    )
+    (property "Footprint" "Package_DIP:DIP-28_W15.24mm" (id 2) (at 210.82 334.01 0)
+      (effects (font (size 1.27 1.27)) hide)
+    )
