File: docs/leo/leo.kicad_sch (KiCad schematic)
At the start: 21 parts, among them IC11 GAL16V8, IC20 74153, IC21 74LS273, IC29 74LS273, IC37 MB81C78A, IC38 MB81C78A, IC40 74LS04, IC41 GAL16V8, IC51 GAL16V8, IC52 74LS32, IC56 74LS245, IC57 74LS245, IC58 74LS244, IC59 74LS244, IC60 74LS244, IC61 74LS139, IC62 74LS20, IC8 7486

Commit message: Finished GA20 pinout Roughed in sound latch, ym2151 and ga20 signals in A board
Other:
- added sheet Audio (audio.kicad_sch)
- note added: "Audio Stuff"
- moved on the sheet: U?C

Commit message: Add ym filters and misinx path Upgrade to kicad 7
Other:
- added sheet Audio Mix (audio_mix.kicad_sch)
